Commit message: Clean up unused legacy robot assets + rename K1_serial → K1_22dof
Drop obsolete asset directories that were superseded by either the
mjlab asset_zoo (T1, Go2) or menagerie (G1) paths and are no longer
referenced by any preset:

- assets/T1/*          — superseded by menagerie_T1 + mjlab booster_t1
- assets/T1_deprecated — old serial/locomotion variants, unused
- assets/go1_*         — Go1 never wired into any preset
- assets/multilink_arms — synthetic test arms, unused

Also rename K1_serial.{urdf,xml} to K1_22dof.{urdf,xml} to match the
naming convention used by T1_23dof / G1_29dof and add/update K1
collision meshes (foot, trunk, head).

Co-Authored-By: Claude Opus 4.7 (1M context) <noreply@anthropic.com>

File: JaxRLWorld/rlworld/assets/K1/K1_22dof-ZED.urdf (robot description, URDF)
Before this commit: robot K1, 23 links, 22 joints
Links:
- link Head_2: mass 0.70 -> 0.781574; geometry collision mesh filename=meshes/Head_2_ZED.STL; visual mesh filename=meshes/Head_2_ZED.STL
Joints:
- joint AAHead_yaw: type fixed -> revolute
- joint ALeft_Shoulder_Pitch: type fixed -> revolute
- joint ARight_Shoulder_Pitch: type fixed -> revolute
- joint Head_pitch: type fixed -> revolute
- joint Left_Elbow_Pitch: type fixed -> revolute
- joint Left_Elbow_Yaw: type fixed -> revolute
- joint Left_Shoulder_Roll: type fixed -> revolute
- joint Right_Elbow_Pitch: type fixed -> revolute
- joint Right_Elbow_Yaw: type fixed -> revolute
- joint Right_Shoulder_Roll: type fixed -> revolute

File: JaxRLWorld/rlworld/assets/K1/K1_22dof.urdf (robot description, URDF)
Before this commit: robot K1, 23 links, 22 joints
Joints:
- joint AAHead_yaw: type fixed -> revolute
- joint ALeft_Shoulder_Pitch: type fixed -> revolute
- joint ARight_Shoulder_Pitch: type fixed -> revolute
- joint Head_pitch: type fixed -> revolute
- joint Left_Elbow_Pitch: type fixed -> revolute
- joint Left_Elbow_Yaw: type fixed -> revolute
- joint Left_Shoulder_Roll: type fixed -> revolute
- joint Right_Elbow_Pitch: type fixed -> revolute
- joint Right_Elbow_Yaw: type fixed -> revolute
- joint Right_Shoulder_Roll: type fixed -> revolute
